File: Adafruit Feather 32u4 RFMxx.brd (EAGLE design)
At the start: 50.8 x 22.9 mm, 40 parts, among them IC1 ATMEGA32U4-MU, SW1 SPST_TACT-KMR2, U2 AP2112-3.3, U3 MCP73831T-2ACI/OT, X1 JSTPH, X2 uFL, X3 microUSB, Y1 8MHz

Commit message: fix broken #8 trace
Connections:
- removed net 8: IC1.28
- net D8_CS: now also IC1.28
Routing:
- net D8_CS: track 47.4 -> 50.6 mm
Changed lines of the file:
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@@
 <?xml version="1.0" encoding="utf-8"?>
 <!DOCTYPE eagle SYSTEM "eagle.dtd">
-<eagle version="6.6.0">
+<eagle version="6.4">
 <drawing>
 <settings>
@@
 <wire x1="50.1015" y1="19.177" x2="49.9745" y2="19.05" width="0.254" layer="1"/>
 <wire x1="49.9745" y1="19.05" x2="49.9745" y2="18.757" width="0.254" layer="1"/>
+<contactref element="IC1" pad="28"/>
+<wire x1="23.5585" y1="17.7165" x2="23.5585" y2="14.524" width="0.254" layer="1"/>
 </signal>
 <signal name="D7_IRQ">
@@
 <contactref element="U4" pad="15P"/>
 </signal>
-<signal name="8">
-<contactref element="IC1" pad="28"/>
-</signal>
 </signals>
