File: Adafruit Feather 32u4 RFMxx.sch (EAGLE design)
At the start: 36 parts, among them IC1 ATMEGA32U4-MU, SW1 SPST_TACT-KMR2, U2 AP2112-3.3, U3 MCP73831T-2ACI/OT, X1 JSTPH, X2 uFL, X3 microUSB, Y1 8MHz

Commit message: fix broken #8 trace
Connections:
- removed net 8: IC1.PB4(ADC11)
- net D8_CS: now also IC1.PB4(ADC11)
Changed lines of the file:
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@@
 <?xml version="1.0" encoding="utf-8"?>
 <!DOCTYPE eagle SYSTEM "eagle.dtd">
-<eagle version="6.6.0">
+<eagle version="6.4">
 <drawing>
 <settings>
@@
 <pinref part="R1" gate="G$1" pin="1"/>
 </segment>
+<segment>
+<wire x1="236.22" y1="127" x2="254" y2="127" width="0.1524" layer="91"/>
+<pinref part="IC1" gate="G$1" pin="PB4(ADC11)"/>
+<label x="238.76" y="127" size="1.778" layer="95"/>
+</segment>
 </net>
 <net name="D7_IRQ" class="0">
@@
 </segment>
 </net>
-<net name="8" class="0">
-<segment>
-<wire x1="236.22" y1="127" x2="254" y2="127" width="0.1524" layer="91"/>
-<pinref part="IC1" gate="G$1" pin="PB4(ADC11)"/>
-<label x="238.76" y="127" size="1.778" layer="95"/>
-</segment>
-</net>
